File: Robko01Apple2Adapter/R01A2A/R01A2A.sch (KiCad schematic (older format))
At the start: 14 parts, among them J1 B, J2 C, U1 2716, U2 74HC00, U3 74HC04, U4 74LS30, U5 i8216, U6 i8226, U7 i8216

Commit message: Change project libraries
Parts:
- removed BUS1: A2_BUS, Apple2:BUS_A2, symbol Apple2:A2_BUS
- added BUS1: A2_BUS, symbol Apple2_bus:A2_BUS
Connections:
- net +5V: now also BUS1.25 (+5V)
- net A0: now also BUS1.2 (A0)
- net A1: now also BUS1.3 (A1)
- net A10: now also BUS1.12 (A10)
- net A15: now also BUS1.17 (A15)
- net A2: now also BUS1.4 (A2)
- net A3: now also BUS1.5 (A3)
- net A4: now also BUS1.6 (A4)
- net A5: now also BUS1.7 (A5)
- net A6: now also BUS1.8 (A6)
- net A7: now also BUS1.9 (A7)
- net A8: now also BUS1.10 (A8)
- net A9: now also BUS1.11 (A9)
- net D0: now also BUS1.49 (D0)
- net D1: now also BUS1.48 (D1)
- net D2: now also BUS1.47 (D2)
- net D3: now also BUS1.46 (D3)
- net D4: now also BUS1.45 (D4)
- net D5: now also BUS1.44 (D5)
- net D6: now also BUS1.43 (D6)
- net D7: now also BUS1.42 (D7)
- net DEVSEL: now also BUS1.41 (~DEVSEL)
- net DMA: now also BUS1.24 (DMA_OUT), BUS1.27 (DMA_IN)
- net GND: now also BUS1.26 (GND)
- net INT: now also BUS1.23 (INT_OUT), BUS1.28 (INT_IN)
- net IO_SEL: now also BUS1.1 (~I/O_SEL)
- net STROBE: now also BUS1.20 (~STROBE)
Changed lines of the file:
@@
 Comment4 ""
 $EndDescr
-$Comp
-L Apple2:A2_BUS BUS1
-U 1 1 5F1C0064
-P 5800 7400
-F 0 "BUS1" H 7200 9487 60  0000 C CNN
-F 1 "A2_BUS" H 7200 9381 60  0000 C CNN
-F 2 "Apple2:BUS_A2" H 5800 7400 60  0001 C CNN
-F 3 "" H 5800 7400 60  0000 C CNN
-	1    5800 7400
-	1    0    0    -1
-$EndComp
 NoConn ~ 6400 7200
 NoConn ~ 6400 7000
@@
 Wire Wire Line
 	17200 5450 17200 6350
-Wire Bus Line
-	2700 5100 2700 7600
-Wire Bus Line
-	4700 5100 4700 7600
-Wire Bus Line
-	5700 5100 5700 10400
-Wire Bus Line
-	9000 5100 9000 8100
-Wire Bus Line
-	8700 5100 8700 10500
 Connection ~ 17200 6350
 Text Label 9150 6400 0    50   ~ 0
@@
 Text Label 8450 10000 0    50   ~ 0
 A1
+Wire Bus Line
+	2700 5100 2700 7600
+Wire Bus Line
+	4700 5100 4700 7600
+Wire Bus Line
+	5700 5100 5700 10400
+Wire Bus Line
+	9000 5100 9000 8100
+Wire Bus Line
+	8700 5100 8700 10500
+$Comp
+L Apple2_bus:A2_BUS BUS1
+U 1 1 5F3CD9AD
+P 5800 7400
+F 0 "BUS1" H 7200 9487 60  0000 C CNN
+F 1 "A2_BUS" H 7200 9381 60  0000 C CNN
+F 2 "" H 5800 7400 60  0000 C CNN
+F 3 "" H 5800 7400 60  0000 C CNN
+	1    5800 7400
+	1    0    0    -1
+$EndComp
 $EndSCHEMATC
